Commit message: Add parallel gripper to robot

File: install/gantry/share/gantry/urdf/parallel_beam_gantry.ros2_control.xacro (robot description, xacro)
@@ -65,4 +65,13 @@
         <state_interface name="velocity"/>
       </joint>
+      <!-- Gripper Joint -->
+      <joint name="left_finger_joint">
+        <command_interface name="position">
+          <param name="min">0</param>
+          <param name="max">0.03</param>
+        </command_interface>
+        <state_interface name="position"/>
+        <state_interface name="velocity"/>
+      </joint>
       <!-- ============================================================================= -->
       <!-- |                         MIMIC JOINT (PASSIVE)                             | -->

File: install/gantry/share/gantry/urdf/parallel_beam_gantry.xacro (robot description, xacro)
@@ -17,4 +17,5 @@
   <xacro:include filename="$(find gantry)/urdf/parallel_beam_gantry.gazebo.xacro"/>
   <xacro:include filename="$(find gantry)/urdf/parallel_beam_gantry.camera.xacro"/>
+  <xacro:include filename="$(find gantry)/urdf/simple_gripper.urdf.xacro"/>
   <!-- =================================================================================== -->
   <!-- |                           INSTANTIATE MACROS                                    | -->
@@ -33,3 +34,8 @@
     </xacro:overhead_rgb_camera>
   </xacro:if>
+  <!-- Instantiate the gripper and attach it to the end effector -->
+  <xacro:simple_gripper name_prefix="" parent_link="end_effector_link">
+    <!-- Attach to the bottom tip of the 0.5m long end effector beam (-0.25m in Z) -->
+    <origin xyz="0 0 -0.25" rpy="0 0 0"/>
+  </xacro:simple_gripper>
 </robot>
