Commit message: adding grasping

File: install/gantry/share/gantry/urdf/parallel_beam_gantry.gazebo.xacro (robot description, xacro)
@@ -8,6 +8,18 @@
     <gazebo>
       <plugin name="gz_ros2_control::GazeboSimROS2ControlPlugin" filename="gz_ros2_control-system">
-        <parameters>$(find gantry_moveit_config)/config/ros2_controllers.yaml</parameters>
+        <parameters>$(find gantry_moveit_config_2)/config/ros2_controllers.yaml</parameters>
       </plugin>
+          <plugin filename="gz-sim-detachable-joint-system" name="gz::sim::systems::DetachableJoint">
+        <!-- 1. The Robot (Parent) -->
+        <!-- <parent_model>parallel_beam_gantry</parent_model> -->
+        <parent_link>z_slider_link</parent_link>
+        <!-- 2. The Object (Child) -->
+        <child_model>sphere_red</child_model>
+        <child_link>link</child_link>
+        <!-- 3. The Signal -->
+        <attach_topic>/gripper/attach</attach_topic>
+        <detach_topic>/gripper/detach</detach_topic>
+        <suppress_child_collision>true</suppress_child_collision>
+    </plugin>
     </gazebo>
     <!-- =============================================================================== -->

File: install/gantry/share/gantry/urdf/parallel_beam_gantry.ros2_control.xacro (robot description, xacro)
@@ -74,4 +74,11 @@
         <state_interface name="velocity"/>
       </joint>
+            <!-- === ADD THIS: MIMIC JOINT (SLAVE) === -->
+      <joint name="right_finger_joint">
+        <param name="mimic">left_finger_joint</param>
+        <param name="multiplier">1</param>
+        <state_interface name="position"/>
+        <state_interface name="velocity"/>
+      </joint>
       <!-- ============================================================================= -->
       <!-- |                         MIMIC JOINT (PASSIVE)                             | -->

File: install/gantry/share/gantry/urdf/simple_gripper.urdf.xacro (robot description, xacro)
@@ -54,9 +54,9 @@
       <child link="${name_prefix}left_finger_link"/>
       <!-- The finger starts offset from the center of the base -->
-      <origin xyz="0 0.045 -0.025" rpy="0 0 0"/>
+      <origin xyz="0 0.01 -0.025" rpy="0 0 0"/>
       <!-- It moves outwards along the positive Y-axis -->
       <axis xyz="0 1 0"/>
       <!-- 'lower=0' is closed, 'upper=0.03' is open -->
-      <limit lower="0.0" upper="0.03" effort="20" velocity="0.5"/>
+      <limit lower="0.0" upper="0.05" effort="20" velocity="0.5"/>
     </joint>
     <!-- Right Finger (Slave) -->
@@ -79,8 +79,8 @@
       <child link="${name_prefix}right_finger_link"/>
       <!-- This finger starts on the opposite side of the base -->
-      <origin xyz="0 -0.045 -0.025" rpy="0 0 0"/>
+      <origin xyz="0 -0.01 -0.025" rpy="0 0 0"/>
       <!-- It moves outwards along the negative Y-axis -->
       <axis xyz="0 -1 0"/>
-      <limit lower="0.0" upper="0.03" effort="20" velocity="0.5"/>
+      <limit lower="0.0" upper="0.05" effort="20" velocity="0.5"/>
       <!-- The MIMIC tag is the key: it makes this joint copy the master joint's value -->
       <mimic joint="${name_prefix}left_finger_joint" multiplier="1" offset="0"/>
